Commit message: try gcs on intermediate trajectories?

File: pete_assets/assets/box.urdf (robot description, URDF)
Before this commit: robot box, 1 links, 0 joints
Links:
- link box_link: geometry collision box size=0.05 3 2; visual box size=0.05 3 2

File: pete_assets/assets/camera_box_big.urdf (robot description, URDF)
Before this commit: robot camera_box_big, 1 links, 0 joints
Links:
- link camera_box_link: geometry collision box size=0.1 0.8 1.2; visual box size=0.1 0.8 1.2

File: pete_assets/assets/camera_box_small.urdf (robot description, URDF)
Before this commit: robot camera_box_small, 1 links, 0 joints
Links:
- link camera_box_link: geometry collision box size=0.3 0.3 0.46; visual box size=0.3 0.3 0.46
